Commit message: Rename packages names

File: alpha_ins_description/urdf/base.urdf.xacro (robot description, xacro)
@@ -1,9 +1,9 @@
 <?xml version="1.0"?>
-<robot name="alpha_std" xmlns:xacro="http://ros.org/wiki/xacro">
+<robot name="alpha_ins" xmlns:xacro="http://ros.org/wiki/xacro">
     <link name="base_link">
         <visual>
             <origin xyz="0.0 -0.63 -0.57" rpy="0.0 0.0 1.5707963"/>
             <geometry>
-                <mesh filename="package://alpha_std_description/mesh/alpha_std.stl" scale="0.001 0.001 0.001"/>
+                <mesh filename="package://alpha_ins_description/mesh/alpha_ins.stl" scale="0.001 0.001 0.001"/>
             </geometry>
         </visual>

File: alpha_ins_stonefish/description/alpha_std.scn.xacro (robot description, xacro)
@@ -8,7 +8,7 @@
 -->
 <scenario xmlns:xacro="http://ros.org/wiki/xacro">
-    <xacro:include filename="$(find alpha_std_stonefish)/description/looks.scn.xacro"/>
-    <xacro:include filename="$(find alpha_std_stonefish)/description/materials.scn.xacro"/>
-    <xacro:macro name="alpha_std" params="xyz rpy robot_name">
+    <xacro:include filename="$(find alpha_ins_stonefish)/description/looks.scn.xacro"/>
+    <xacro:include filename="$(find alpha_ins_stonefish)/description/materials.scn.xacro"/>
+    <xacro:macro name="alpha_ins" params="xyz rpy robot_name">
         <robot name="${robot_name}" fixed="false" self_collisions="false">
             <base_link name="Vehicle" type="compound" physics="submerged">

File: alpha_ins_stonefish/scenarios/ocean.scn.xacro (robot description, xacro)
@@ -9,6 +9,6 @@
 <scenario xmlns:xacro="http://ros.org/wiki/xacro">
     <xacro:arg name="robot_name" default="changeme"/>
-    <xacro:include filename="$(find alpha_std_stonefish)/description/alpha_std.scn.xacro"/>
-    <xacro:alpha_std robot_name="$(arg robot_name)" xyz="0.0 0.0 0.0" rpy="0.0 0.0 0.0"/>
+    <xacro:include filename="$(find alpha_ins_stonefish)/description/alpha_ins.scn.xacro"/>
+    <xacro:alpha_ins robot_name="$(arg robot_name)" xyz="0.0 0.0 0.0" rpy="0.0 0.0 0.0"/>
     <environment>
         <ned latitude="41" longitude="-71"/>

File: alpha_ins_stonefish/scenarios/tank.scn.xacro (robot description, xacro)
@@ -9,5 +9,5 @@
 <scenario xmlns:xacro="http://ros.org/wiki/xacro">
     <xacro:arg name="robot_name" default="changeme"/>
-    <xacro:include filename="$(find alpha_std_stonefish)/description/alpha_std.scn.xacro"/>
+    <xacro:include filename="$(find alpha_ins_stonefish)/description/alpha_ins.scn.xacro"/>
     <xacro:alpha_sci robot_name="$(arg robot_name)" xyz="0.0 0.0 0.0" rpy="0.0 0.0 0.0"/>
     <environment>

Commit message: Rename and add base description

File: alpha_ins_description/urdf/base.urdf.xacro (robot description, xacro)
@@ -58,4 +58,17 @@
         <child link="surge_thruster_link"/>
     </joint>
+    <!-- new front-facing thrusters -->
+    <link name="front_left_thruster_link"/>
+    <joint name="front_left_thruster_joint" type="continuous">
+        <origin xyz="0.0 0.1 0.0" rpy="0.0 0.0 0.0"/>
+        <parent link="base_link"/>
+        <child link="front_left_thruster_link"/>
+    </joint>
+    <link name="front_right_thruster_link"/>
+    <joint name="front_right_thruster_joint" type="continuous">
+        <origin xyz="0.0 -0.1 0.0" rpy="0.0 0.0 0.0"/>
+        <parent link="base_link"/>
+        <child link="front_right_thruster_link"/>
+    </joint>
     <link name="heave_bow_thruster_link"/>
     <joint name="heave_bow_thruster_joint" type="fixed">

File: alpha_ins_stonefish/description/alpha_ins.scn.xacro (robot description, xacro)
@@ -5,5 +5,5 @@
     Email: emircem@uri.edu;emircem.gezer@gmail.com
     Year: 2022
-    Copyright (C) 2022 Smart Ocean Systems Laboratory
+    Copyright (C) 2023 Smart Ocean Systems Laboratory
 -->
 <scenario xmlns:xacro="http://ros.org/wiki/xacro">
@@ -78,4 +78,30 @@
             </joint>
             <!--  -->
+           <!-- Add new thrusters at the front of the vehicle -->
+            <link name="FrontLeftThruster" type="box" physics="submerged">
+                <dimensions xyz="0.1 0.02 0.02"/> <!-- Adjust dimensions as needed -->
+                <origin xyz="-1.0 0.1 0.0" rpy="0.0 0.0 0.0"/> <!-- Adjust position as needed -->
+                <material name="Neutral"/>
+                <look name="Black"/> <!-- Adjust color as needed -->
+            </link>
+            <link name="FrontRightThruster" type="box" physics="submerged">
+                <dimensions xyz="0.1 0.02 0.02"/> <!-- Adjust dimensions as needed -->
+                <origin xyz="-1.0 -0.1 0.0" rpy="0.0 0.0 0.0"/> <!-- Adjust position as needed -->
+                <material name="Neutral"/>
+                <look name="Black"/> <!-- Adjust color as needed -->
+            </link>
+            <!-- Add joints for the servo-controlled thrusters -->
+            <joint name="FrontLeftThrusterJoint" type="continuous">
+                <parent link="Vehicle"/>
+                <child link="FrontLeftThruster"/>
+                <origin rpy="0.0 0.0 0.0" xyz="-1.0 0.1 0.0"/> <!-- Adjust position as needed -->
+                <axis xyz="0.0 0.0 1.0"/>
+            </joint>
+            <joint name="FrontRightThrusterJoint" type="continuous">
+                <parent link="Vehicle"/>
+                <child link="FrontRightThruster"/>
+                <origin rpy="0.0 0.0 0.0" xyz="-1.0 -0.1 0.0"/> <!-- Adjust position as needed -->
+                <axis xyz="0.0 0.0 1.0"/>
+            </joint>
             <actuator name="ThrusterSwayBow" type="thruster">
                 <link name="Base"/>

Commit message: adding surge servos 1

File: alpha_ins_description/urdf/base.urdf.xacro (robot description, xacro)
@@ -59,5 +59,5 @@
     </joint>
     <!-- new front-facing thrusters -->
-    <link name="front_left_thruster_link"/>
+    <!-- <link name="front_left_thruster_link"/>
     <joint name="front_left_thruster_joint" type="continuous">
         <origin xyz="0.0 0.1 0.0" rpy="0.0 0.0 0.0"/>
@@ -70,5 +70,5 @@
         <parent link="base_link"/>
         <child link="front_right_thruster_link"/>
-    </joint>
+    </joint> -->
     <link name="heave_bow_thruster_link"/>
     <joint name="heave_bow_thruster_joint" type="fixed">

File: alpha_ins_stonefish/description/alpha_ins.scn.xacro (robot description, xacro)
@@ -78,30 +78,82 @@
             </joint>
             <!--  -->
-           <!-- Add new thrusters at the front of the vehicle -->
-            <link name="FrontLeftThruster" type="box" physics="submerged">
-                <dimensions xyz="0.1 0.02 0.02"/> <!-- Adjust dimensions as needed -->
-                <origin xyz="-1.0 0.1 0.0" rpy="0.0 0.0 0.0"/> <!-- Adjust position as needed -->
-                <material name="Neutral"/>
-                <look name="Black"/> <!-- Adjust color as needed -->
+            <!-- Start: Starboard Surge -->
+            <link name="ThrusterSurgeStarboardDuct" type="compound" physics="submerged">
+                <external_part name="SurgeStarboardDuct" type="model" physics="submerged" buoyant="true">
+                    <physical>
+                        <mesh filename="duct_reduced.obj" scale="0.001"/>
+                        <origin rpy="0.0 0.0 0.0" xyz="0.0 0.0 0.0"/>
+                    </physical>
+                    <visual>
+                        <mesh filename="duct.obj" scale="0.001"/>
+                        <origin rpy="0.0 0.0 0.0" xyz="0.0 0.0 0.0"/>
+                    </visual>
+                    <material name="Neutral"/>
+                    <look name="black"/>
+                    <compound_transform rpy="0.0 -1.57 0.0" xyz="0.0 0.0 0.0"/>
+                </external_part>
             </link>
-            <link name="FrontRightThruster" type="box" physics="submerged">
-                <dimensions xyz="0.1 0.02 0.02"/> <!-- Adjust dimensions as needed -->
-                <origin xyz="-1.0 -0.1 0.0" rpy="0.0 0.0 0.0"/> <!-- Adjust position as needed -->
-                <material name="Neutral"/>
-                <look name="Black"/> <!-- Adjust color as needed -->
+            <actuator name="ThrusterSurgeStarboard" type="thruster">
+                <link name="ThrusterSurgeStarboardDuct"/>
+                <origin rpy="0.0 0.0 0.0" xyz="0.0 0.0 0.0"/>
+                <specs thrust_coeff="0.4315" thrust_coeff_backward="0.3404" torque_coeff="0.01" max_rpm="3000.0"/>
+                <propeller diameter="0.08" right="true">
+                    <mesh filename="prop.obj" scale="1.0"/>
+                    <material name="Neutral"/>
+                    <look name="white"/>
+                </propeller>
+                <ros_subscriber topic="/${robot_name}/control/thruster/surge_starboard"/>
+            </actuator>
+            <joint name="surge_starboard_joint" type="revolute">
+                <parent name="Vehicle"/>
+                <child name="ThrusterSurgeStarboardDuct"/>
+                <origin rpy="0.0 0.0 0.0" xyz="-1.0956 0.165 0.0"/>
+                <axis xyz="0.0 1.0 0.0"/>
+                <limits min="-1.5705" max="1.5705"/>
+            </joint>
+            <actuator name="ServoStarboardPort" type="servo">
+                <joint name="surge_starboard_joint"/>
+                <controller position_gain="1.1" velocity_gain="0.1" max_torque="10.0"/>
+            </actuator>
+            <!-- End: Starboard Surge -->
+            <!-- Start: Port Surge -->
+            <link name="ThrusterSurgePortDuct" type="compound" physics="submerged">
+                <external_part name="SurgePortDuct" type="model" physics="submerged" buoyant="true">
+                    <physical>
+                        <mesh filename="duct_reduced.obj" scale="0.001"/>
+                        <origin rpy="0.0 0.0 0.0" xyz="0.0 0.0 0.0"/>
+                    </physical>
+                    <visual>
+                        <mesh filename="duct.obj" scale="0.001"/>
+                        <origin rpy="0.0 0.0 0.0" xyz="0.0 0.0 0.0"/>
+                    </visual>
+                    <material name="Neutral"/>
+                    <look name="black"/>
+                    <compound_transform rpy="0.0 -1.57 0.0" xyz="0.0 0.0 0.0"/>
+                </external_part>
             </link>
-            <!-- Add joints for the servo-controlled thrusters -->
-            <joint name="FrontLeftThrusterJoint" type="continuous">
-                <parent link="Vehicle"/>
-                <child link="FrontLeftThruster"/>
-                <origin rpy="0.0 0.0 0.0" xyz="-1.0 0.1 0.0"/> <!-- Adjust position as needed -->
-                <axis xyz="0.0 0.0 1.0"/>
+            <actuator name="ThrusterSurgePort" type="thruster">
+                <link name="ThrusterSurgePortDuct"/>
+                <origin rpy="0.0 0.0 0.0" xyz="0.0 0.0 0.0"/>
+                <specs thrust_coeff="0.4315" thrust_coeff_backward="0.3404" torque_coeff="0.01" max_rpm="3000.0"/>
+                <propeller diameter="0.08" right="true">
+                    <mesh filename="prop.obj" scale="1.0"/>
+                    <material name="Neutral"/>
+                    <look name="white"/>
+                </propeller>
+                <ros_subscriber topic="/${robot_name}/control/thruster/surge_port"/>
+            </actuator>
+            <joint name="surge_port_joint" type="revolute">
+                <parent name="Vehicle"/>
+                <child name="ThrusterSurgePortDuct"/>
+                <origin rpy="0.0 0.0 0.0" xyz="-1.0956 -0.165 0.0"/>
+                <axis xyz="0.0 1.0 0.0"/>
+                <limits min="-1.5705" max="1.5705"/>
             </joint>
-            <joint name="FrontRightThrusterJoint" type="continuous">
-                <parent link="Vehicle"/>
-                <child link="FrontRightThruster"/>
-                <origin rpy="0.0 0.0 0.0" xyz="-1.0 -0.1 0.0"/> <!-- Adjust position as needed -->
-                <axis xyz="0.0 0.0 1.0"/>
-            </joint>
+            <actuator name="ServoSurgePort" type="servo">
+                <joint name="surge_port_joint"/>
+                <controller position_gain="1.1" velocity_gain="0.1" max_torque="10.0"/>
+            </actuator>
+            <!-- End: Port Surge -->
             <actuator name="ThrusterSwayBow" type="thruster">
                 <link name="Base"/>

Commit message: Add Azimuth Thrusters

File: alpha_ins_description/urdf/base.urdf.xacro (robot description, xacro)
@@ -58,4 +58,16 @@
         <child link="surge_thruster_link"/>
     </joint>
+    <link name="surge_port_thruster_link"/>
+    <joint name="surge_port_thruster_joint" type="continuous">
+        <origin xyz="-0.24045 -0.165 0.0" rpy="0.0 0.0 0.0"/>
+        <parent link="base_link"/>
+        <child link="surge_port_thruster_link"/>
+    </joint>
+    <link name="surge_starboard_thruster_link"/>
+    <joint name="surge_starboard_thruster_joint" type="continuous">
+        <origin xyz="-0.24045 0.165 0.0" rpy="0.0 0.0 0.0"/>
+        <parent link="base_link"/>
+        <child link="surge_starboard_thruster_link"/>
+    </joint>
     <!-- new front-facing thrusters -->
     <!-- <link name="front_left_thruster_link"/>

File: alpha_ins_stonefish/description/alpha_ins.scn.xacro (robot description, xacro)
@@ -6,5 +6,5 @@
     Year: 2022
     Copyright (C) 2023 Smart Ocean Systems Laboratory
--->
+    -->
 <scenario xmlns:xacro="http://ros.org/wiki/xacro">
     <xacro:include filename="$(find alpha_ins_stonefish)/description/looks.scn.xacro"/>
@@ -50,5 +50,5 @@
                     <compound_transform rpy="0.0 0.0 0.0" xyz="0.0 0.0 0.0"/>
                 </external_part>
-                <external_part name="ThrusterDuctSurge" type="model" physics="submerged" buoyant="false">
+                <!-- <external_part name="ThrusterDuctSurge" type="model" physics="submerged" buoyant="false">
                     <physical>
                         <mesh filename="duct.obj" scale="0.0015"/>
@@ -62,5 +62,5 @@
                     <look name="black"/>
                     <compound_transform rpy="0.0 0.0 0.0" xyz="0.0 0.0 0.0"/>
-                </external_part>
+                </external_part> -->
             </base_link>
             <!-- the actual base frame  -->
@@ -77,4 +77,38 @@
                 <axis xyz="1.0 0.0 0.0"/>
             </joint>
+            <!-- <external_part name="AzimuthThruster" type="compound" physics="submerged">
+                <origin xyz="-1.325 0.0 0.0" rpy="0.0 0.0 0.0"/>
+                <joint name="AzimuthJoint" type="revolute">
+                    <axis xyz="0.0 0.0 1.0"/>
+                    <origin xyz="0.0 0.0 0.0" rpy="0.0 0.0 0.0"/>
+                    <limit lower="-3.141592653589793" upper="3.141592653589793" effort="100.0" velocity="1.0"/>
+                    <ros_subscriber topic="/${robot_name}/control/azimuth"/>
+                </joint>
+                <link name="ThrusterDuctSurge" type="model" physics="submerged" buoyant="false">
+                    <physical>
+                        <mesh filename="duct.obj" scale="0.0015"/>
+                        <origin rpy="0.0 1.571 0.0" xyz="0.0 0.0 0.0"/>
+                    </physical>
+                    <visual>
+                        <mesh filename="duct.obj" scale="0.0015"/>
+                        <origin rpy="0.0 1.571 0.0" xyz="0.0 0.0 0.0"/>
+                    </visual>
+                    <material name="Neutral"/>
+                    <look name="black"/>
+                    <compound_transform rpy="0.0 0.0 0.0" xyz="0.0 0.0 0.0"/>
+                </link>
+                <actuator name="ThrusterSurge" type="thruster">
+                    <link name="ThrusterDuctSurge"/>
+                    <origin rpy="0.0 0.0 0.0" xyz="0.0 0.0 0.0"/>
+                    <specs thrust_coeff="1.7568" thrust_coeff_backward="1.0882" torque_coeff="0.01" max_rpm="3000.0"/>
+                    <propeller diameter="0.08" right="true">
+                        <origin rpy="1.571 0.0 0.0" xyz="0.0 0.0 0.0"/>
+                        <mesh filename="prop.obj" scale="1.5"/>
+                        <material name="Neutral"/>
+                        <look name="white"/>
+                    </propeller>
+                    <ros_subscriber topic="/${robot_name}/control/thruster/surge"/>
+                </actuator>
+            </external_part> -->
             <!--  -->
             <!-- Start: Starboard Surge -->
@@ -116,4 +150,5 @@
                 <controller position_gain="1.1" velocity_gain="0.1" max_torque="10.0"/>
             </actuator>
+            <ros_joint_subscriber joint_name="surge_starboard_joint" topic="/${robot_name}/joint/servo/starboard" control_mode="position" />
             <!-- End: Starboard Surge -->
             <!-- Start: Port Surge -->
@@ -150,9 +185,10 @@
                 <axis xyz="0.0 1.0 0.0"/>
                 <limits min="-1.5705" max="1.5705"/>
-            </joint>
+                </joint>
             <actuator name="ServoSurgePort" type="servo">
                 <joint name="surge_port_joint"/>
                 <controller position_gain="1.1" velocity_gain="0.1" max_torque="10.0"/>
             </actuator>
+            <ros_joint_subscriber joint_name="surge_port_joint" topic="/${robot_name}/joint/servo/port" control_mode="position" />
             <!-- End: Port Surge -->
             <actuator name="ThrusterSwayBow" type="thruster">
@@ -189,5 +225,5 @@
                 <ros_subscriber topic="/${robot_name}/control/thruster/heave_bow"/>
             </actuator>
-            <actuator name="ThrusterSurge" type="thruster">
+            <!-- <actuator name="ThrusterSurge" type="thruster">
                 <link name="Base"/>
                 <origin rpy="0.0 0.0 0.0" xyz="-1.325 0.0 0.0"/>
@@ -200,5 +236,5 @@
                 </propeller>
                 <ros_subscriber topic="/${robot_name}/control/thruster/surge"/>
-            </actuator>
+            </actuator> -->
             <sensor name="pressure" type="pressure" rate="5.0">
                 <link name="Base"/>
